File: October Launch Avionics.sch (KiCad schematic (older format))
At the start: 20 parts, among them IC1 MPU-6050, IC2 790, IC3 BMP384, J1 U.FL-R-SMT_01_, J2 MEM2075-00-140-01-A, U1 ESP32-WROOM-32D

Commit message: updated reference designators
Parts:
- gave numbers to parts that had none: 2
Connections:
- no-connect marks 26 -> 27
Changed lines of the file:
@@
 NoConn ~ 7800 4950
 $Comp
-L power:+3.3V #PWR?
+L power:+3.3V #PWR025
 U 1 1 61080F74
 P 9800 1950
-F 0 "#PWR?" H 9800 1800 50  0001 C CNN
+F 0 "#PWR025" H 9800 1800 50  0001 C CNN
 F 1 "+3.3V" H 9750 2100 50  0000 C CNN
 F 2 "" H 9800 1950 50  0001 C CNN
@@
 EN
 $Comp
-L SamacSys_Parts:PTS645SM43JSMTR92_LFS S?
+L SamacSys_Parts:PTS645SM43JSMTR92_LFS S1
 U 1 1 61081AFF
 P 9350 5850
-F 0 "S?" H 9950 6115 50  0000 C CNN
+F 0 "S1" H 9950 6115 50  0000 C CNN
 F 1 "PTS645SM43JSMTR92_LFS" H 9950 6024 50  0000 C CNN
 F 2 "PTS645SM43JSMTR92LFS" H 10400 5950 50  0001 L CNN
@@
 $EndComp
 $Comp
-L power:GND #PWR?
+L power:GND #PWR024
 U 1 1 61083EA1
 P 9350 5950
-F 0 "#PWR?" H 9350 5700 50  0001 C CNN
+F 0 "#PWR024" H 9350 5700 50  0001 C CNN
 F 1 "GND" H 9355 5777 50  0000 C CNN
 F 2 "" H 9350 5950 50  0001 C CNN
@@
 EN
 $Comp
-L Device:R R?
+L Device:R R5
 U 1 1 61088122
 P 9050 5700
-F 0 "R?" H 9120 5746 50  0000 L CNN
+F 0 "R5" H 9120 5746 50  0000 L CNN
 F 1 "330" H 9120 5655 50  0000 L CNN
 F 2 "" V 8980 5700 50  0001 C CNN
@@
 $EndComp
 $Comp
-L power:+3.3V #PWR?
+L power:+3.3V #PWR023
 U 1 1 61088AE9
 P 9050 5550
-F 0 "#PWR?" H 9050 5400 50  0001 C CNN
+F 0 "#PWR023" H 9050 5400 50  0001 C CNN
 F 1 "+3.3V" H 9000 5700 50  0000 C CNN
 F 2 "" H 9050 5550 50  0001 C CNN
@@
 Wire Wire Line
 	9050 5850 9350 5850
+NoConn ~ 1300 4550
 $EndSCHEMATC

Commit message: Wired up ESP-32 with USB C and UART Chip
- Connected the ESP-32 to the CP2102N chip
- Connected the CP2102N chip to USB type C port
- Wired up connections as per the datasheet:
https://www.snapeda.com/parts/CP2102N-A01-GQFN20R/Silicon%20Labs/datasheet/
Parts:
- added D?: SP0503BAHT, Package_TO_SOT_SMD:SOT-143, symbol Power_Protection:SP0503BAHT
- added P?: USB_C_Plug_USB2.0, symbol Connector:USB_C_Plug_USB2.0
- added R?: 22.1k, symbol Device:R
- added R?: 47.5k, symbol Device:R
- added U?: CP2102N-A01-GQFN20R, SILABS_QFN20, symbol CP2102N-A01-GQFN20R:CP2102N-A01-GQFN20R
- C1, C2, C3, C4, C5, C6: symbol Device:C -> October-Launch-Avionics-rescue:C-Device
- D1, D2: symbol Device:LED -> October-Launch-Avionics-rescue:LED-Device
- R1, R2, R3, R4, R5: symbol Device:R -> October-Launch-Avionics-rescue:R-Device
- U1: symbol RF_Module:ESP32-WROOM-32D -> October-Launch-Avionics-rescue:ESP32-WROOM-32D-RF_Module
Connections:
- net labels added: D+, D-, Earth, VBUS
- wire segments 46 -> 73
- no-connect marks 27 -> 41

Commit message: Some small changes
Connections:
- net labels added: UART_RX, UART_TX
- net labels removed: Earth
- wire segments 73 -> 61
- no-connect marks 41 -> 42
Other:
- moved on the sheet: D?, R?
Changed lines of the file:
@@
 	1    0    0    -1
 $EndComp
-Wire Wire Line
-	7100 3250 7100 2950
-Wire Wire Line
-	6900 3250 6900 3150
-Wire Wire Line
-	9500 2550 9500 2950
-Wire Wire Line
-	9500 2950 10300 2950
-Wire Wire Line
-	10300 2950 10300 3300
-Wire Wire Line
-	9000 4700 7900 4700
-Wire Wire Line
-	7900 4700 7900 4500
 Wire Notes Line
 	10950 6250 10950 800
@@
 Text GLabel 9700 3300 1    50   Input ~ 0
 D-
-Wire Wire Line
-	10200 3100 10200 3300
-Wire Wire Line
-	9300 3100 10200 3100
-Wire Wire Line
-	9300 2550 9300 3100
-Wire Wire Line
-	6700 4500 7900 4500
 Text GLabel 9800 3300 1    50   Input ~ 0
 D+
-Text GLabel 7850 3700 1    50   Input ~ 0
+Text GLabel 7300 3700 1    50   Input ~ 0
 D+
-$Comp
-L Power_Protection:SP0503BAHT D?
-U 1 1 611016B0
-P 7950 4050
-F 0 "D?" H 8155 4096 50  0000 L CNN
-F 1 "SP0503BAHT" H 8155 4005 50  0000 L CNN
-F 2 "Package_TO_SOT_SMD:SOT-143" H 8175 4000 50  0001 L CNN
-F 3 "http://www.littelfuse.com/~/media/files/littelfuse/technical%20resources/documents/data%20sheets/sp05xxba.pdf" H 8075 4175 50  0001 C CNN
-	1    7950 4050
-	1    0    0    -1
-$EndComp
-$Comp
-L power:Earth #PWR?
-U 1 1 61105D3A
-P 7950 4400
-F 0 "#PWR?" H 7950 4150 50  0001 C CNN
-F 1 "Earth" H 7950 4250 50  0001 C CNN
-F 2 "" H 7950 4400 50  0001 C CNN
-F 3 "~" H 7950 4400 50  0001 C CNN
-	1    7950 4400
-	1    0    0    -1
-$EndComp
-Text GLabel 8050 3000 2    50   Input ~ 0
+Text GLabel 7300 3000 1    50   Input ~ 0
 VBUS
 NoConn ~ 9500 3300
@@
 NoConn ~ 7300 3300
 NoConn ~ 7300 3200
-Text GLabel 7950 3500 1    50   Input ~ 0
+Text GLabel 7300 3500 1    50   Input ~ 0
 D-
-Wire Wire Line
-	7300 3000 8050 3000
-Wire Wire Line
-	8050 3000 8050 3850
-Wire Wire Line
-	7950 3500 7300 3500
-Wire Wire Line
-	7950 3500 7950 3850
-Wire Wire Line
-	7300 3700 7850 3700
-Wire Wire Line
-	7850 3850 7850 3700
-Wire Wire Line
-	7950 4250 7950 4400
 NoConn ~ 10000 3300
 NoConn ~ 10100 3300
-Text GLabel 9150 4950 0    50   Input ~ 0
+Text GLabel 10200 5150 0    50   Input ~ 0
 VBUS
 Wire Wire Line
-	9650 5250 9650 4950
+	10300 5150 10400 5150
 Wire Wire Line
-	9900 5250 9650 5250
+	10300 4700 10300 5150
+$Comp
+L Device:R R?
+U 1 1 610C423B
+P 10550 5150
+F 0 "R?" V 10343 5150 50  0000 C CNN
+F 1 "47.5k" V 10434 5150 50  0000 C CNN
+F 2 "" V 10480 5150 50  0001 C CNN
+F 3 "~" H 10550 5150 50  0001 C CNN
+	1    10550 5150
+	0    1    1    0
+$EndComp
 Wire Wire Line
-	10700 5250 10800 5250
-Wire Wire Line
-	10300 5250 10400 5250
-Wire Wire Line
-	10300 5250 10200 5250
-Connection ~ 10300 5250
-Wire Wire Line
-	10300 4700 10300 5250
+	10200 4700 10200 4800
+$Comp
+L October-Launch-Avionics-rescue:GND-power #PWR?
+U 1 1 610AB54E
+P 9000 4700
+F 0 "#PWR?" H 9000 4450 50  0001 C CNN
+F 1 "GND" H 9005 4527 50  0000 C CNN
+F 2 "" H 9000 4700 50  0001 C CNN
+F 3 "" H 9000 4700 50  0001 C CNN
+	1    9000 4700
+	1    0    0    -1
+$EndComp
+$Comp
+L October-Launch-Avionics-rescue:GND-power #PWR?
+U 1 1 610ADFD1
+P 6700 4500
+F 0 "#PWR?" H 6700 4250 50  0001 C CNN
+F 1 "GND" H 6705 4327 50  0000 C CNN
+F 2 "" H 6700 4500 50  0001 C CNN
+F 3 "" H 6700 4500 50  0001 C CNN
+	1    6700 4500
+	1    0    0    -1
+$EndComp
 $Comp
 L Device:R R?
 U 1 1 610C2020
-P 10050 5250
-F 0 "R?" V 9843 5250 50  0000 C CNN
-F 1 "22.1k" V 9934 5250 50  0000 C CNN
-F 2 "" V 9980 5250 50  0001 C CNN
-F 3 "~" H 10050 5250 50  0001 C CNN
-	1    10050 5250
-	0    1    1    0
+P 10200 4950
+F 0 "R?" V 9993 4950 50  0000 C CNN
+F 1 "22.1k" V 10084 4950 50  0000 C CNN
+F 2 "" V 10130 4950 50  0001 C CNN
+F 3 "~" H 10200 4950 50  0001 C CNN
+	1    10200 4950
+	1    0    0    -1
+$EndComp
+Wire Wire Line
+	10200 5100 10200 5150
+Wire Wire Line
+	10300 5150 10200 5150
+Connection ~ 10300 5150
+$Comp
+L October-Launch-Avionics-rescue:GND-power #PWR?
+U 1 1 610BD0D9
+P 10750 5200
+F 0 "#PWR?" H 10750 4950 50  0001 C CNN
+F 1 "GND" H 10755 5027 50  0000 C CNN
+F 2 "" H 10750 5200 50  0001 C CNN
+F 3 "" H 10750 5200 50  0001 C CNN
+	1    10750 5200
+	1    0    0    -1
+$EndComp
+Wire Wire Line
+	10750 5200 10750 5150
+Wire Wire Line
+	10750 5150 10700 5150
+NoConn ~ 10550 5950
+Text GLabel 9300 2550 3    50   Input ~ 0
+UART_TX
+Text GLabel 9500 2550 3    50   Input ~ 0
+UART_RX
+Text GLabel 10200 3300 1    50   Input ~ 0
+UART_TX
+Text GLabel 10300 3300 1    50   Input ~ 0
+UART_RX
+$Comp
+L October-Launch-Avionics-rescue:GND-power #PWR?
+U 1 1 610AAC9B
+P 7900 3650
+F 0 "#PWR?" H 7900 3400 50  0001 C CNN
+F 1 "GND" H 7905 3477 50  0000 C CNN
+F 2 "" H 7900 3650 50  0001 C CNN
+F 3 "" H 7900 3650 50  0001 C CNN
+	1    7900 3650
+	1    0    0    -1
 $EndComp
 $Comp
-L Device:R R?
-U 1 1 610C423B
-P 10550 5250
-F 0 "R?" V 10343 5250 50  0000 C CNN
-F 1 "47.5k" V 10434 5250 50  0000 C CNN
-F 2 "" V 10480 5250 50  0001 C CNN
-F 3 "~" H 10550 5250 50  0001 C CNN
-	1    10550 5250
-	0    1    1    0
-$EndComp
-$Comp
-L power:Earth #PWR?
-U 1 1 610C5906
-P 10800 5250
-F 0 "#PWR?" H 10800 5000 50  0001 C CNN
-F 1 "Earth" H 10800 5100 50  0001 C CNN
-F 2 "" H 10800 5250 50  0001 C CNN
-F 3 "~" H 10800 5250 50  0001 C CNN
-	1    10800 5250
+L Power_Protection:SP0503BAHT D?
+U 1 1 611016B0
+P 7650 3600
+F 0 "D?" H 7855 3646 50  0000 L CNN
+F 1 "SP0503BAHT" H 7855 3555 50  0000 L CNN
+F 2 "Package_TO_SOT_SMD:SOT-143" H 7875 3550 50  0001 L CNN
+F 3 "http://www.littelfuse.com/~/media/files/littelfuse/technical%20resources/documents/data%20sheets/sp05xxba.pdf" H 7775 3725 50  0001 C CNN
+	1    7650 3600
 	0    -1   -1   0
 $EndComp
 Wire Wire Line
-	10200 4700 10200 4950
+	7900 3650 7900 3600
 Wire Wire Line
-	10200 4950 9650 4950
-Connection ~ 9650 4950
+	7900 3600 7850 3600
 Wire Wire Line
-	9650 4950 9150 4950
+	7300 3700 7450 3700
+Wire Wire Line
+	7300 3500 7400 3500
+Wire Wire Line
+	7400 3500 7400 3600
+Wire Wire Line
+	7400 3600 7450 3600
+Wire Wire Line
+	7300 3000 7450 3000
+Wire Wire Line
+	7450 3000 7450 3500
 $EndSCHEMATC
