File: October Launch Avionics.sch (KiCad schematic (older format))
At the start: 30 parts, among them IC1 MPU-6050, IC2 790, IC3 BMP384, J1 U.FL-R-SMT_01_, J2 MEM2075-00-140-01-A, U1 ESP32-WROOM-32D, U2 LM2596S-5

Commit message: Fixed some merging weirdness?
Parts:
- removed C7, C8: CP, symbol Device:CP
- removed D3: D, symbol Device:D
- removed L1: L, symbol Device:L
- removed U2: LM2596S-5, Package_TO_SOT_SMD:TO-263-5_TabPin3, symbol Regulator_Switching:LM2596S-5
Changed lines of the file:
@@
 	6000 800  6000 6250
 Wire Notes Line
-	10700 800  6000 800
+	10950 800  6000 800
 Text Notes 8000 750  0    50   ~ 0
 Teency & Peripherals
@@
 	10950 6250 10950 800
 Wire Notes Line
-	6000 6250 10700 6250
+	6000 6250 10950 6250
 Text GLabel 9700 3300 1    50   Input ~ 0
 D-
@@
 Wire Wire Line
 	7450 3000 7450 3500
-$Comp
-L Regulator_Switching:LM2596S-5 U2
-U 1 1 61015F13
-P 2800 1250
-F 0 "U2" H 2800 1617 50  0000 C CNN
-F 1 "LM2596S-5" H 2800 1526 50  0000 C CNN
-F 2 "Package_TO_SOT_SMD:TO-263-5_TabPin3" H 2850 1000 50  0001 L CIN
-F 3 "http://www.ti.com/lit/ds/symlink/lm2596.pdf" H 2800 1250 50  0001 C CNN
-	1    2800 1250
-	1    0    0    -1
-$EndComp
-$Comp
-L power:+5V #PWR0107
-U 1 1 6102E3B5
-P 4150 1150
-F 0 "#PWR0107" H 4150 1000 50  0001 C CNN
-F 1 "+5V" V 4165 1278 50  0000 L CNN
-F 2 "" H 4150 1150 50  0001 C CNN
-F 3 "" H 4150 1150 50  0001 C CNN
-	1    4150 1150
-	0    1    1    0
-$EndComp
-$Comp
-L Device:L L1
-U 1 1 610792E4
-P 3500 1350
-F 0 "L1" V 3690 1350 50  0000 C CNN
-F 1 "L" V 3599 1350 50  0000 C CNN
-F 2 "" H 3500 1350 50  0001 C CNN
-F 3 "~" H 3500 1350 50  0001 C CNN
-	1    3500 1350
-	0    -1   -1   0
-$EndComp
-$Comp
-L Device:D D3
-U 1 1 61076105
-P 3350 1500
-F 0 "D3" V 3304 1580 50  0000 L CNN
-F 1 "D" V 3395 1580 50  0000 L CNN
-F 2 "" H 3350 1500 50  0001 C CNN
-F 3 "~" H 3350 1500 50  0001 C CNN
-	1    3350 1500
-	0    1    1    0
-$EndComp
-Connection ~ 3350 1650
-$Comp
-L power:GND #PWR0105
-U 1 1 61028B2E
-P 1600 1650
-F 0 "#PWR0105" H 1600 1400 50  0001 C CNN
-F 1 "GND" V 1605 1522 50  0000 R CNN
-F 2 "" H 1600 1650 50  0001 C CNN
-F 3 "" H 1600 1650 50  0001 C CNN
-	1    1600 1650
-	0    1    1    0
-$EndComp
-Wire Wire Line
-	2300 1350 2300 1650
-Connection ~ 2300 1650
-Wire Wire Line
-	2300 1650 2800 1650
-Wire Wire Line
-	2800 1550 2800 1650
-Connection ~ 2800 1650
-Wire Wire Line
-	2800 1650 3350 1650
-Wire Wire Line
-	3300 1350 3350 1350
-Connection ~ 3350 1350
-Wire Wire Line
-	3650 1350 3700 1350
-Wire Wire Line
-	3700 1350 3700 1150
-Connection ~ 3700 1150
-Wire Wire Line
-	3700 1150 3300 1150
-Wire Wire Line
-	3700 1150 4150 1150
-$Comp
-L power:GND #PWR0106
-U 1 1 610A5901
-P 4100 1650
-F 0 "#PWR0106" H 4100 1400 50  0001 C CNN
-F 1 "GND" V 4105 1522 50  0000 R CNN
-F 2 "" H 4100 1650 50  0001 C CNN
-F 3 "" H 4100 1650 50  0001 C CNN
-	1    4100 1650
-	0    -1   -1   0
-$EndComp
-$Comp
-L Device:CP C8
-U 1 1 610A7BB2
-P 3700 1500
-F 0 "C8" H 3818 1546 50  0000 L CNN
-F 1 "CP" H 3818 1455 50  0000 L CNN
-F 2 "" H 3738 1350 50  0001 C CNN
-F 3 "~" H 3700 1500 50  0001 C CNN
-	1    3700 1500
-	1    0    0    -1
-$EndComp
-Wire Wire Line
-	3350 1650 3700 1650
-Connection ~ 3700 1350
-Connection ~ 3700 1650
-Wire Wire Line
-	3700 1650 4100 1650
-$Comp
-L Device:CP C7
-U 1 1 610AC176
-P 2050 1400
-F 0 "C7" H 2168 1446 50  0000 L CNN
-F 1 "CP" H 2168 1355 50  0000 L CNN
-F 2 "" H 2088 1250 50  0001 C CNN
-F 3 "~" H 2050 1400 50  0001 C CNN
-	1    2050 1400
-	1    0    0    -1
-$EndComp
-Wire Wire Line
-	1600 1150 2050 1150
-Wire Wire Line
-	1600 1650 2050 1650
-Wire Wire Line
-	2050 1250 2050 1150
-Connection ~ 2050 1150
-Wire Wire Line
-	2050 1150 2300 1150
-Wire Wire Line
-	2050 1550 2050 1650
-Connection ~ 2050 1650
-Wire Wire Line
-	2050 1650 2300 1650
 $EndSCHEMATC

Commit message: Update October Launch Avionics.sch
Parts:
- added C10: CP 10uF, symbol Device:CP
- added C7: CP 1mF, symbol Device:CP
- added C8: CP 220uF, symbol Device:CP
- added C9: CP 1uF, symbol Device:CP
- added D3: D, symbol Device:D
- added L1: L, symbol Device:L
- added U2: LM2596S-5, Package_TO_SOT_SMD:TO-263-5_TabPin3, symbol Regulator_Switching:LM2596S-5
- added U3: TPS78533QWDRBRQ1, Package_TO_SOT_SMD:SOT-23-5, symbol Regulator_Linear:TPS78218DDC
- gave numbers to parts that had none: 5
Connections:
- net +3V3: now also C10.2
- net GND: now also C7.2, C8.2, D3.2 (A), U2.3 (GND), U2.5 (~ON~/OFF), U3.2 (GND), U3.4 (GND)
- new net: C7.1, U2.1 (VIN)
- new net: D3.1 (K), L1.1, U2.2 (OUT)
- new net: C9.2, U3.1 (IN)
- new net: C10.1, U3.5 (OUT)
- new net +5V: C8.1, C9.1, L1.2, U2.4 (FB)
Changed lines of the file:
@@
 NoConn ~ 1300 4550
 $Comp
-L CP2102N-A01-GQFN20R:CP2102N-A01-GQFN20R U?
+L CP2102N-A01-GQFN20R:CP2102N-A01-GQFN20R U4
 U 1 1 610661BB
 P 9700 4000
-F 0 "U?" H 9700 4967 50  0000 C CNN
+F 0 "U4" H 9700 4967 50  0000 C CNN
 F 1 "CP2102N-A01-GQFN20R" H 9700 4876 50  0000 C CNN
 F 2 "SILABS_QFN20" H 9700 4000 50  0001 L BNN
@@
 $EndComp
 $Comp
-L Connector:USB_C_Plug_USB2.0 P?
+L Connector:USB_C_Plug_USB2.0 P1
 U 1 1 61091D25
 P 6700 3600
-F 0 "P?" H 6807 4467 50  0000 C CNN
+F 0 "P1" H 6807 4467 50  0000 C CNN
 F 1 "USB_C_Plug_USB2.0" H 6807 4376 50  0000 C CNN
 F 2 "" H 6850 3600 50  0001 C CNN
@@
 	10300 4700 10300 5150
 $Comp
-L Device:R R?
+L Device:R R7
 U 1 1 610C423B
 P 10550 5150
-F 0 "R?" V 10343 5150 50  0000 C CNN
+F 0 "R7" V 10343 5150 50  0000 C CNN
 F 1 "47.5k" V 10434 5150 50  0000 C CNN
 F 2 "" V 10480 5150 50  0001 C CNN
@@
 	10200 4700 10200 4800
 $Comp
-L October-Launch-Avionics-rescue:GND-power #PWR?
+L October-Launch-Avionics-rescue:GND-power #PWR0108
 U 1 1 610AB54E
 P 9000 4700
-F 0 "#PWR?" H 9000 4450 50  0001 C CNN
+F 0 "#PWR0108" H 9000 4450 50  0001 C CNN
 F 1 "GND" H 9005 4527 50  0000 C CNN
 F 2 "" H 9000 4700 50  0001 C CNN
@@
 $EndComp
 $Comp
-L October-Launch-Avionics-rescue:GND-power #PWR?
+L October-Launch-Avionics-rescue:GND-power #PWR0109
 U 1 1 610ADFD1
 P 6700 4500
-F 0 "#PWR?" H 6700 4250 50  0001 C CNN
+F 0 "#PWR0109" H 6700 4250 50  0001 C CNN
 F 1 "GND" H 6705 4327 50  0000 C CNN
 F 2 "" H 6700 4500 50  0001 C CNN
@@
 $EndComp
 $Comp
-L Device:R R?
+L Device:R R6
 U 1 1 610C2020
 P 10200 4950
-F 0 "R?" V 9993 4950 50  0000 C CNN
+F 0 "R6" V 9993 4950 50  0000 C CNN
 F 1 "22.1k" V 10084 4950 50  0000 C CNN
 F 2 "" V 10130 4950 50  0001 C CNN
@@
 Connection ~ 10300 5150
 $Comp
-L October-Launch-Avionics-rescue:GND-power #PWR?
+L October-Launch-Avionics-rescue:GND-power #PWR0110
 U 1 1 610BD0D9
 P 10750 5200
-F 0 "#PWR?" H 10750 4950 50  0001 C CNN
+F 0 "#PWR0110" H 10750 4950 50  0001 C CNN
 F 1 "GND" H 10755 5027 50  0000 C CNN
 F 2 "" H 10750 5200 50  0001 C CNN
@@
 UART_RX
 $Comp
-L October-Launch-Avionics-rescue:GND-power #PWR?
+L October-Launch-Avionics-rescue:GND-power #PWR0111
 U 1 1 610AAC9B
 P 7900 3650
-F 0 "#PWR?" H 7900 3400 50  0001 C CNN
+F 0 "#PWR0111" H 7900 3400 50  0001 C CNN
 F 1 "GND" H 7905 3477 50  0000 C CNN
 F 2 "" H 7900 3650 50  0001 C CNN
@@
 $EndComp
 $Comp
-L Power_Protection:SP0503BAHT D?
+L Power_Protection:SP0503BAHT D4
 U 1 1 611016B0
 P 7650 3600
-F 0 "D?" H 7855 3646 50  0000 L CNN
+F 0 "D4" H 7855 3646 50  0000 L CNN
 F 1 "SP0503BAHT" H 7855 3555 50  0000 L CNN
 F 2 "Package_TO_SOT_SMD:SOT-143" H 7875 3550 50  0001 L CNN
@@
 Wire Wire Line
 	7450 3000 7450 3500
+$Comp
+L Regulator_Switching:LM2596S-5 U2
+U 1 1 61015F13
+P 2800 1250
+F 0 "U2" H 2800 1617 50  0000 C CNN
+F 1 "LM2596S-5" H 2800 1526 50  0000 C CNN
+F 2 "Package_TO_SOT_SMD:TO-263-5_TabPin3" H 2850 1000 50  0001 L CIN
+F 3 "http://www.ti.com/lit/ds/symlink/lm2596.pdf" H 2800 1250 50  0001 C CNN
+	1    2800 1250
+	1    0    0    -1
+$EndComp
+$Comp
+L power:+5V #PWR0107
+U 1 1 6102E3B5
+P 4150 1150
+F 0 "#PWR0107" H 4150 1000 50  0001 C CNN
+F 1 "+5V" V 4165 1278 50  0000 L CNN
+F 2 "" H 4150 1150 50  0001 C CNN
+F 3 "" H 4150 1150 50  0001 C CNN
+	1    4150 1150
+	0    1    1    0
+$EndComp
+$Comp
+L Device:L L1
+U 1 1 610792E4
+P 3500 1350
+F 0 "L1" V 3690 1350 50  0000 C CNN
+F 1 "L" V 3599 1350 50  0000 C CNN
+F 2 "" H 3500 1350 50  0001 C CNN
+F 3 "~" H 3500 1350 50  0001 C CNN
+	1    3500 1350
+	0    -1   -1   0
+$EndComp
+$Comp
+L Device:D D3
+U 1 1 61076105
+P 3350 1500
+F 0 "D3" V 3304 1580 50  0000 L CNN
+F 1 "D" V 3395 1580 50  0000 L CNN
+F 2 "" H 3350 1500 50  0001 C CNN
+F 3 "~" H 3350 1500 50  0001 C CNN
+	1    3350 1500
+	0    1    1    0
+$EndComp
+Connection ~ 3350 1650
+$Comp
+L power:GND #PWR0105
+U 1 1 61028B2E
+P 1600 1650
+F 0 "#PWR0105" H 1600 1400 50  0001 C CNN
+F 1 "GND" V 1605 1522 50  0000 R CNN
+F 2 "" H 1600 1650 50  0001 C CNN
+F 3 "" H 1600 1650 50  0001 C CNN
+	1    1600 1650
+	0    1    1    0
+$EndComp
+Wire Wire Line
+	2300 1350 2300 1650
+Connection ~ 2300 1650
+Wire Wire Line
+	2300 1650 2800 1650
+Wire Wire Line
+	2800 1550 2800 1650
+Connection ~ 2800 1650
+Wire Wire Line
+	2800 1650 3350 1650
+Wire Wire Line
+	3300 1350 3350 1350
+Connection ~ 3350 1350
+Wire Wire Line
+	3650 1350 3700 1350
+Wire Wire Line
+	3700 1350 3700 1150
+Connection ~ 3700 1150
+Wire Wire Line
+	3700 1150 3300 1150
+Wire Wire Line
+	3700 1150 4150 1150
+$Comp
+L power:GND #PWR0106
+U 1 1 610A5901
+P 4100 1650
+F 0 "#PWR0106" H 4100 1400 50  0001 C CNN
+F 1 "GND" V 4105 1522 50  0000 R CNN
+F 2 "" H 4100 1650 50  0001 C CNN
+F 3 "" H 4100 1650 50  0001 C CNN
+	1    4100 1650
+	0    -1   -1   0
+$EndComp
+$Comp
+L Device:CP C8
+U 1 1 610A7BB2
+P 3700 1500
+F 0 "C8" H 3818 1546 50  0000 L CNN
+F 1 "CP 220uF" H 3818 1455 50  0000 L CNN
+F 2 "" H 3738 1350 50  0001 C CNN
+F 3 "~" H 3700 1500 50  0001 C CNN
+	1    3700 1500
+	1    0    0    -1
+$EndComp
+Wire Wire Line
+	3350 1650 3700 1650
+Connection ~ 3700 1350
+Connection ~ 3700 1650
+Wire Wire Line
+	3700 1650 4100 1650
+Wire Wire Line
+	1600 1150 2050 1150
+Connection ~ 2050 1150
+Wire Wire Line
+	2050 1150 2300 1150
+$Comp
+L Device:CP C7
+U 1 1 610AC176
+P 2050 1500
+F 0 "C7" H 2168 1546 50  0000 L CNN
+F 1 "CP 1mF" H 2168 1455 50  0000 L CNN
+F 2 "" H 2088 1350 50  0001 C CNN
+F 3 "~" H 2050 1500 50  0001 C CNN
+	1    2050 1500
+	1    0    0    -1
+$EndComp
+Wire Wire Line
+	1600 1650 2050 1650
+Connection ~ 2050 1650
+Wire Wire Line
+	2050 1650 2300 1650
+Wire Wire Line
+	2050 1150 2050 1350
+$Comp
+L Regulator_Linear:TPS78218DDC U3
+U 1 1 6112307C
+P 2800 2200
+F 0 "U3" H 2800 2567 50  0000 C CNN
+F 1 "TPS78533QWDRBRQ1" H 2800 2476 50  0000 C CNN
+F 2 "Package_TO_SOT_SMD:SOT-23-5" H 2800 2550 50  0001 C CNN
+F 3 "http://www.ti.com/lit/gpn/tps782" H 2800 2700 50  0001 C CNN
+	1    2800 2200
+	1    0    0    -1
+$EndComp
+$Comp
+L power:GND #PWR0112
+U 1 1 61128578
+P 2800 2500
+F 0 "#PWR0112" H 2800 2250 50  0001 C CNN
+F 1 "GND" H 2805 2327 50  0000 C CNN
+F 2 "" H 2800 2500 50  0001 C CNN
+F 3 "" H 2800 2500 50  0001 C CNN
+	1    2800 2500
+	1    0    0    -1
+$EndComp
+$Comp
+L Device:CP C10
+U 1 1 61127C7D
+P 3250 2100
+F 0 "C10" V 3400 2100 50  0000 C CNN
+F 1 "CP  10uF" V 3100 2050 50  0000 C CNN
+F 2 "" H 3288 1950 50  0001 C CNN
+F 3 "~" H 3250 2100 50  0001 C CNN
+	1    3250 2100
+	0    -1   -1   0
+$EndComp
+$Comp
+L power:+3.3V #PWR0113
+U 1 1 61129D40
+P 3400 2100
+F 0 "#PWR0113" H 3400 1950 50  0001 C CNN
+F 1 "+3.3V" V 3415 2228 50  0000 L CNN
+F 2 "" H 3400 2100 50  0001 C CNN
+F 3 "" H 3400 2100 50  0001 C CNN
+	1    3400 2100
+	0    1    1    0
+$EndComp
+$Comp
+L Device:CP C9
+U 1 1 61125B0C
+P 2350 2100
+F 0 "C9" V 2500 2100 50  0000 C CNN
+F 1 "CP  1uF" V 2200 2100 50  0000 C CNN
+F 2 "" H 2388 1950 50  0001 C CNN
+F 3 "~" H 2350 2100 50  0001 C CNN
+	1    2350 2100
+	0    -1   -1   0
+$EndComp
+$Comp
+L power:+5V #PWR0114
+U 1 1 61128D00
+P 2200 2100
+F 0 "#PWR0114" H 2200 1950 50  0001 C CNN
+F 1 "+5V" V 2215 2228 50  0000 L CNN
+F 2 "" H 2200 2100 50  0001 C CNN
+F 3 "" H 2200 2100 50  0001 C CNN
+	1    2200 2100
+	0    -1   -1   0
+$EndComp
 $EndSCHEMATC
