File: _autosave-October Launch Avionics.sch (KiCad schematic (older format))
At the start: 28 parts, among them IC1 MPU-6050, IC2 790, IC3 BMP384, J1 U.FL-R-SMT_01_, J2 MEM2075-00-140-01-A, J3 Conn_01x04_Male, J4 Conn_01x04_Male, J5 Conn_01x02_Male, U1 ESP32-WROOM-32D, U2 LM2596S-5

Commit message: Added Molex Connectors
Hopefully correctly
Parts:
- added J?: Micro Molex 5 Pin - I2C, symbol Connector:Conn_01x05_Male
- added J?: Mirco Molex 5 Pin SPI, symbol Connector:Conn_01x05_Male
- added J?: Molex-Con - Cam, Connector_Molex:Molex_CLIK-Mate_502386-0470_1x04-1MP_P1.25mm_Horizontal, symbol Connector:Conn_01x04_Male
- J3: value Conn_01x04_Male -> Molex Micro 4 Pin #2
- J4: value Conn_01x04_Male -> Molex Mirco 4 Pin #1
- J5: value Conn_01x02_Male -> Molex Mirco 2 Pin
Connections:
- net labels added: +3.3VA, +5VA, Cam_RX, Cam_TX, Spare_CS, Spare_SCL, Spare_SCLK, Spare_SDA, Spare_SDI, Spare_SDO
Other:
- moved on the sheet: J3, J4, J5
